Commit message: Add: env

File: urdf/kuka_iiwa/modified_model.urdf (robot description, URDF)
Before this commit: robot lbr_iiwa, 14 links, 13 joints
Joints:
- joint tcp_joint: origin xyz=0 0 0 rpy=0 0 0 -> xyz=0.0 -0.4 -0.2 rpy=0 0 0

Commit message: Add: reward

File: urdf/kuka_iiwa/modified_model.urdf (robot description, URDF)
Before this commit: robot lbr_iiwa, 14 links, 13 joints
Joints:
- joint tcp_joint: origin xyz=0.0 -0.4 -0.2 rpy=0 0 0 -> xyz=0 0 -0.1 rpy=0 0 0

Commit message: Debug

File: urdf/kuka_iiwa/modified_model.urdf (robot description, URDF)
Before this commit: robot lbr_iiwa, 14 links, 13 joints
Joints:
- joint tcp_joint: origin xyz=0 0 -0.1 rpy=0 0 0 -> xyz=0.0 -0.4 -0.2 rpy=0 0 0

Commit message: Debug

File: urdf/kuka_iiwa/modified_model.urdf (robot description, URDF)
Before this commit: robot lbr_iiwa, 14 links, 13 joints
Joints:
- joint tcp_joint: origin xyz=0 0 -0.1 rpy=0 0 0 -> xyz=0 0 0 rpy=0 0 0

Commit message: Debug: robot

File: urdf/kuka_iiwa/modified_model.urdf (robot description, URDF)
Before this commit: robot lbr_iiwa, 14 links, 13 joints
Joints:
- joint lbr_iiwa_joint_3: type revolute -> fixed
- joint tcp_joint: origin xyz=0 0 0 rpy=0 0 0 -> xyz=0.0 0.0 -0.15 rpy=0.0 0.0 0.0
