Commit message: Debug: robot

File: urdf/kuka_iiwa_6/basic_model.urdf (robot description, URDF)
Before this commit: robot lbr_iiwa, 14 links, 13 joints
Links:
- removed link lbr_iiwa_link_2
- removed link lbr_iiwa_link_3
- removed link lbr_iiwa_link_4
- removed link lbr_iiwa_link_5
- removed link lbr_iiwa_link_6
- removed link lbr_iiwa_link_7
- removed link marker_origin
- removed link marker_x
- removed link marker_y
- removed link marker_z
- removed link tcp_link
- removed link world_link
- added link lbr_iiwa_link_23, mass 4; collision mesh filename=meshes/link_23.stl; visual mesh filename=meshes/link_23.stl
Joints:
- removed joint connector_origin
- removed joint lbr_iiwa_joint_2
- removed joint lbr_iiwa_joint_3
- removed joint lbr_iiwa_joint_4
- removed joint lbr_iiwa_joint_5
- removed joint lbr_iiwa_joint_6
- removed joint lbr_iiwa_joint_7
- removed joint marker_origin_x
- removed joint marker_origin_y
- removed joint marker_origin_z
- removed joint tcp_joint
- removed joint world_joint
- added joint lbr_iiwa_joint_23: type revolute, parent lbr_iiwa_link_1, child lbr_iiwa_link_23, origin xyz=0 0 0.2025 rpy=1.57079632679   0 3.14159265359, axis 0 0 1, limit lower=-2.09439510239 upper=2.09439510239 effort=300 velocity=10

Commit message: Add: robot

File: urdf/kuka_iiwa_6/basic_model.urdf (robot description, URDF)
Before this commit: robot lbr_iiwa, 3 links, 2 joints
Links:
- added link lbr_iiwa_link_4, mass 2.7; collision mesh filename=meshes/link_4.stl; visual mesh filename=meshes/link_4.stl
- added link lbr_iiwa_link_5, mass 1.7; collision mesh filename=meshes/link_5.stl; visual mesh filename=meshes/link_5.stl
- added link lbr_iiwa_link_6, mass 1.8; collision mesh filename=meshes/link_6.stl; visual mesh filename=meshes/link_6.obj
- added link lbr_iiwa_link_7, mass 0.3; collision mesh filename=meshes/link_7.stl; visual mesh filename=meshes/link_7.obj
- added link marker_origin, mass 0.001; visual box size=0.002 0.002 0.002
- added link marker_x, mass 0.001; visual box size=0.005 0.001 0.001
- added link marker_y, mass 0.001; visual box size=0.001 0.005 0.001
- added link marker_z, mass 0.001; visual box size=0.001 0.001 0.005
Joints:
- added joint connector_origin: type fixed, parent lbr_iiwa_link_7, child marker_origin, origin xyz=0.0 0.0 0.045 rpy=0 0 0
- added joint lbr_iiwa_joint_4: type revolute, parent lbr_iiwa_link_23, child lbr_iiwa_link_4, origin xyz=0.42 0 0 rpy=3.14159265359 0 0, axis 0 0 1, limit lower=-2.09439510239 upper=2.09439510239 effort=300 velocity=10
- added joint lbr_iiwa_joint_5: type revolute, parent lbr_iiwa_link_4, child lbr_iiwa_link_5, origin xyz=0 0.1845 0 rpy=-1.57079632679 3.14159265359 0, axis 0 0 1, limit lower=-2.96705972839 upper=2.96705972839 effort=300 velocity=10
- added joint lbr_iiwa_joint_6: type revolute, parent lbr_iiwa_link_5, child lbr_iiwa_link_6, origin xyz=0 0 0.2155 rpy=1.57079632679 0 0, axis 0 0 1, limit lower=-2.09439510239 upper=2.09439510239 effort=300 velocity=10
- added joint lbr_iiwa_joint_7: type revolute, parent lbr_iiwa_link_6, child lbr_iiwa_link_7, origin xyz=0 0.081 0 rpy=-1.57079632679 3.14159265359 0, axis 0 0 1, limit lower=-3.05432619099 upper=3.05432619099 effort=300 velocity=10
- added joint marker_origin_x: type fixed, parent marker_origin, child marker_x, origin xyz=0.005 0.0 0.0 rpy=0 0 0
- added joint marker_origin_y: type fixed, parent marker_origin, child marker_y, origin xyz=0.0 0.005 0.0 rpy=0 0 0
- added joint marker_origin_z: type fixed, parent marker_origin, child marker_z, origin xyz=0.0 0.0 0.005 rpy=0 0 0
- joint lbr_iiwa_joint_23: origin xyz=0 0 0.2025 rpy=1.57079632679   0 3.14159265359 -> xyz=0 0 0.2025 rpy=-1.57079632679   0 0

Commit message: DEbug: robot

File: urdf/kuka_iiwa_6/basic_model.urdf (robot description, URDF)
Before this commit: robot lbr_iiwa, 11 links, 10 joints
Links:
- added link tcp_link, mass 0.001; visual box size=0.002 0.002 0.002
- added link world_link, mass 0.001; visual box size=0.002 0.002 0.002
Joints:
- added joint tcp_joint: type fixed, parent world_link, child tcp_link, origin xyz=0 0 0 rpy=0 0 0, axis 0 0 1
- added joint world_joint: type fixed, parent lbr_iiwa_link_7, child world_link, origin xyz=0 0 0.045 rpy=0 3.14159265359 0, axis 0 0 1
- joint connector_origin: origin xyz=0.0 0.0 0.045 rpy=0 0 0 -> xyz=0.0 0.0 0 rpy=0 0 0; parent lbr_iiwa_link_7 -> tcp_link

File: urdf/kuka_iiwa_6/modified_model.urdf (robot description, URDF)
Before this commit: robot lbr_iiwa, 14 links, 13 joints
Links:
- removed link lbr_iiwa_link_2
- removed link lbr_iiwa_link_3
- added link lbr_iiwa_link_23, mass 4; collision mesh filename=meshes/link_23.stl; visual mesh filename=meshes/link_23.stl
- link lbr_iiwa_link_4: geometry collision mesh filename=meshes/link_4.stl; visual mesh filename=meshes/link_4.stl
- link lbr_iiwa_link_5: geometry collision mesh filename=meshes/link_5.stl; visual mesh filename=meshes/link_5.stl
Joints:
- removed joint lbr_iiwa_joint_2
- removed joint lbr_iiwa_joint_3
- added joint lbr_iiwa_joint_23: type revolute, parent lbr_iiwa_link_1, child lbr_iiwa_link_23, origin xyz=0 0 0.2025 rpy=-1.57079632679   0 0, axis 0 0 1, limit lower=-2.09439510239 upper=2.09439510239 effort=300 velocity=10
- joint connector_origin: origin xyz=0.0 0.0 0.0 rpy=0 0 0 -> xyz=0.0 0.0 0 rpy=0 0 0
- joint lbr_iiwa_joint_4: origin xyz=0 0 0.2155 rpy=1.57079632679 0 0 -> xyz=0.42 0 0 rpy=3.14159265359 0 0; parent lbr_iiwa_link_3 -> lbr_iiwa_link_23
- joint marker_origin_x: origin xyz=0.0025 0.0 0.0 rpy=0 0 0 -> xyz=0.005 0.0 0.0 rpy=0 0 0
- joint marker_origin_y: origin xyz=0.0 0.0025 0.0 rpy=0 0 0 -> xyz=0.0 0.005 0.0 rpy=0 0 0
- joint marker_origin_z: origin xyz=0.0 0.0 0.0025 rpy=0 0 0 -> xyz=0.0 0.0 0.005 rpy=0 0 0
- joint tcp_joint: origin xyz=0 0 0 rpy=0 0 0 -> xyz=0 0 -0.05 rpy=0 0 0

Commit message: Debug: robot

File: urdf/kuka_iiwa_6/basic_model.urdf (robot description, URDF)
Before this commit: robot lbr_iiwa, 13 links, 12 joints
Links:
- link marker_x: geometry visual box size=0.01 0.001 0.001
- link marker_y: geometry visual box size=0.001 0.01 0.001
- link marker_z: geometry visual box size=0.001 0.001 0.01

File: urdf/kuka_iiwa_6/modified_model.urdf (robot description, URDF)
Before this commit: robot lbr_iiwa, 13 links, 12 joints
Links:
- link marker_x: geometry visual box size=0.01 0.001 0.001
- link marker_y: geometry visual box size=0.001 0.01 0.001
- link marker_z: geometry visual box size=0.001 0.001 0.01
Joints:
- joint tcp_joint: origin xyz=0 0 -0.05 rpy=0 0 0 -> xyz=0 0 0 rpy=0 0 0

Commit message: Debug: robot

File: urdf/kuka_iiwa_6/basic_model.urdf (robot description, URDF)
Before this commit: robot lbr_iiwa, 13 links, 12 joints
Links:
- link lbr_iiwa_link_0: geometry collision mesh filename=meshes/link_0_mod.stl; visual mesh filename=meshes/link_0_mod.stl
- link lbr_iiwa_link_1: geometry collision mesh filename=meshes/link_1_mod.stl; visual mesh filename=meshes/link_1_mod.stl
- link lbr_iiwa_link_23: geometry collision mesh filename=meshes/link_23_mod.stl; visual mesh filename=meshes/link_23_mod.stl
- link lbr_iiwa_link_4: geometry collision mesh filename=meshes/link_4_mod.stl; visual mesh filename=meshes/link_4_mod.stl
- link lbr_iiwa_link_5: geometry collision mesh filename=meshes/link_5_mod.stl; visual mesh filename=meshes/link_5_mod.stl
- link lbr_iiwa_link_6: geometry collision mesh filename=meshes/link_6_mod.stl; visual mesh filename=meshes/link_6_mod.stl
- link lbr_iiwa_link_7: geometry collision mesh filename=meshes/link_7_mod.stl; visual mesh filename=meshes/link_7_mod.stl
Joints:
- joint lbr_iiwa_joint_23: axis 0 0 1 -> 0 1 0; limit lower=-2.09439510239 upper=2.09439510239 effort=300 velocity=10 -> lower=-2.99439510239 upper=2.99439510239 effort=300 velocity=10; origin xyz=0 0 0.2025 rpy=-1.57079632679   0 0 -> xyz=0 0 0.2025 rpy=0 0 0
- joint lbr_iiwa_joint_4: axis 0 0 1 -> 0 1 0; limit lower=-2.09439510239 upper=2.09439510239 effort=300 velocity=10 -> lower=-2.99439510239 upper=4.99439510239 effort=300 velocity=10; origin xyz=0.42 0 0 rpy=3.14159265359 0 0 -> xyz=0.42 0 0 rpy=0 0 0
- joint lbr_iiwa_joint_5: limit lower=-2.96705972839 upper=2.96705972839 effort=300 velocity=10 -> lower=-5.96705972839 upper=5.96705972839 effort=300 velocity=15; origin xyz=0 0.1845 0 rpy=-1.57079632679 3.14159265359 0 -> xyz=0 0 0.4 rpy=0 0 0
- joint lbr_iiwa_joint_6: axis 0 0 1 -> 0 1 0; limit lower=-2.09439510239 upper=2.09439510239 effort=300 velocity=10 -> lower=-2.09439510239 upper=2.09439510239 effort=300 velocity=15; origin xyz=0 0 0.2155 rpy=1.57079632679 0 0 -> xyz=0 0 0 rpy=0 0 0
- joint lbr_iiwa_joint_7: limit lower=-3.05432619099 upper=3.05432619099 effort=300 velocity=10 -> lower=-3.05432619099 upper=3.05432619099 effort=300 velocity=15; origin xyz=0 0.081 0 rpy=-1.57079632679 3.14159265359 0 -> xyz=0 0 0.126 rpy=0 0 0
- joint world_joint: origin xyz=0 0 0.045 rpy=0 3.14159265359 0 -> xyz=0 0 0 rpy=0 3.14159265359 0

File: urdf/kuka_iiwa_6/modified_model.urdf (robot description, URDF)
Before this commit: robot lbr_iiwa, 13 links, 12 joints
Links:
- link lbr_iiwa_link_0: geometry collision mesh filename=meshes/link_0_mod.stl; visual mesh filename=meshes/link_0_mod.stl
- link lbr_iiwa_link_1: geometry collision mesh filename=meshes/link_1_mod.stl; visual mesh filename=meshes/link_1_mod.stl
- link lbr_iiwa_link_23: geometry collision mesh filename=meshes/link_23_mod.stl; visual mesh filename=meshes/link_23_mod.stl
- link lbr_iiwa_link_4: geometry collision mesh filename=meshes/link_4_mod.stl; visual mesh filename=meshes/link_4_mod.stl
- link lbr_iiwa_link_5: geometry collision mesh filename=meshes/link_5_mod.stl; visual mesh filename=meshes/link_5_mod.stl
- link lbr_iiwa_link_6: geometry collision mesh filename=meshes/link_6_mod.stl; visual mesh filename=meshes/link_6_mod.stl
- link lbr_iiwa_link_7: geometry collision mesh filename=meshes/link_7_mod.stl; visual mesh filename=meshes/link_7_mod.stl
Joints:
- joint lbr_iiwa_joint_23: axis 0 0 1 -> 0 1 0; limit lower=-2.09439510239 upper=2.09439510239 effort=300 velocity=10 -> lower=-2.99439510239 upper=2.99439510239 effort=300 velocity=10; origin xyz=0 0 0.2025 rpy=-1.57079632679   0 0 -> xyz=0 0 0.2025 rpy=0 0 0
- joint lbr_iiwa_joint_4: axis 0 0 1 -> 0 1 0; limit lower=-2.09439510239 upper=2.09439510239 effort=300 velocity=10 -> lower=-2.99439510239 upper=4.99439510239 effort=300 velocity=10; origin xyz=0.42 0 0 rpy=3.14159265359 0 0 -> xyz=0.42 0 0 rpy=0 0 0
- joint lbr_iiwa_joint_5: limit lower=-2.96705972839 upper=2.96705972839 effort=300 velocity=10 -> lower=-5.96705972839 upper=5.96705972839 effort=300 velocity=15; origin xyz=0 0.1845 0 rpy=-1.57079632679 3.14159265359 0 -> xyz=0 0 0.4 rpy=0 0 0
- joint lbr_iiwa_joint_6: axis 0 0 1 -> 0 1 0; limit lower=-2.09439510239 upper=2.09439510239 effort=300 velocity=10 -> lower=-2.09439510239 upper=2.09439510239 effort=300 velocity=15; origin xyz=0 0 0.2155 rpy=1.57079632679 0 0 -> xyz=0 0 0 rpy=0 0 0
- joint lbr_iiwa_joint_7: limit lower=-3.05432619099 upper=3.05432619099 effort=300 velocity=10 -> lower=-3.05432619099 upper=3.05432619099 effort=300 velocity=15; origin xyz=0 0.081 0 rpy=-1.57079632679 3.14159265359 0 -> xyz=0 0 0.126 rpy=0 0 0
- joint tcp_joint: origin xyz=0 0.1 0 rpy=-0.3 0.4 0.2 -> xyz=0.0 0.0 -0.15 rpy=0.0 0.0 0.0
- joint world_joint: origin xyz=0 0 0.045 rpy=0 3.14159265359 0 -> xyz=0 0 0 rpy=0 3.14159265359 0

Commit message: Debug: robot

File: urdf/kuka_iiwa_6/basic_model.urdf (robot description, URDF)
Before this commit: robot lbr_iiwa, 13 links, 12 joints
Links:
- link tcp_link: geometry collision box size=0.002 0.002 0.002; visual box size=0.002 0.002 0.002

File: urdf/kuka_iiwa_6/modified_model.urdf (robot description, URDF)
Before this commit: robot lbr_iiwa, 13 links, 12 joints
Links:
- link tcp_link: geometry collision box size=0.002 0.002 0.002; visual box size=0.002 0.002 0.002

Commit message: Debug: Robot

File: urdf/kuka_iiwa_6/basic_model.urdf (robot description, URDF)
Before this commit: robot lbr_iiwa, 13 links, 12 joints
Links:
- link lbr_iiwa_link_0: mass 0.0 -> 10.0
- link lbr_iiwa_link_23: mass 4 -> 8

File: urdf/kuka_iiwa_6/modified_model.urdf (robot description, URDF)
Before this commit: robot lbr_iiwa, 13 links, 12 joints
Links:
- link lbr_iiwa_link_0: mass 0.0 -> 10.0
- link lbr_iiwa_link_23: mass 4 -> 8
